File: Hardware/tinygs_2g4station-main/Board_Tinysgs_2.4GHz_V1/_autosave-Board_ESP_MikroBus_V1.kicad_pcb (KiCad board)
At the start: 2 copper layers, 95.9 x 90.2 mm, 25 parts, among them U1 ESP32-DEVKITC-32D

Commit message: In this branch there will be some alternative routing that isn't useful for now but for the future it may helps
Routing:
- net NSS_0: track 77.1 -> 4.12 mm
- net INT_1: track 91.1 -> 159.9 mm
- net SCK_0: track 121.9 -> 54.7 mm
- net MISO_0: track 118.0 -> 65.0 mm
- net UART0_Rx: track 63.2 -> 17.2 mm
- net I2C_SCL: track 128.8 -> 83.7 mm
- net I2C_SDA: track 128.0 -> 87.3 mm
- net UART2_Rx: track 84.3 -> 51.4 mm
- net UART2_Tx: track 90.5 -> 58.0 mm
- net UART0_Tx: track 61.1 -> 28.5 mm
- net MOSI_0: track 111.4 -> 79.0 mm
- net PWM_1: track 70.2 -> 98.8 mm
- net /33: track 32.6 -> 57.3 mm
- net /34: track 33.0 -> 54.1 mm
- net NSS_1: track 72.7 -> 90.2 mm
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