File: Hardware/2U-PCB-OBC_L476RG/OBS_L476RG/_autosave-OBS_L476RG.kicad_sch (KiCad schematic)
At the start: 7 parts, among them J1 Bus Standard, J2 Micro_SD_Card_Det_Hirose_DM3AT, U2 NUCLEO_L476RG

Commit message: The board is ready. Some verifications required
Connections:
- net Vb: no longer names the net of J1.5 (V_B)
- net Vb: no longer U2.33 (VBAT)
- no-connect marks 55 -> 57
Changed lines of the file:
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@@
   (no_connect (at 162.56 52.07))
   (no_connect (at 120.65 69.85))
+  (no_connect (at 226.06 62.23))
   (no_connect (at 226.06 64.77))
+  (no_connect (at 120.65 120.65))
   (no_connect (at 252.73 72.39))
   (no_connect (at 248.92 59.69))
@@
     (stroke (width 0) (type default))
   )
-  (wire (pts (xy 104.14 120.65) (xy 120.65 120.65))
-    (stroke (width 0) (type default))
-  )
   (wire (pts (xy 252.73 74.93) (xy 248.92 74.93))
     (stroke (width 0) (type default))
@@
     (stroke (width 0) (type default))
   )
-  (wire (pts (xy 222.25 62.23) (xy 226.06 62.23))
-    (stroke (width 0) (type default))
-  )
   (wire (pts (xy 180.34 105.41) (xy 162.56 105.41))
     (stroke (width 0) (type default))
@@
     (effects (font (size 1.27 1.27)) (justify left bottom))
   )
-  (label "Vb" (at 222.25 62.23 180) (fields_autoplaced)
-    (effects (font (size 1.27 1.27)) (justify right bottom))
-  )
   (label "P21" (at 99.06 118.11 180) (fields_autoplaced)
     (effects (font (size 1.27 1.27)) (justify right bottom))
@@
     (effects (font (size 1.27 1.27)) (justify left bottom))
   )
-  (label "Vb" (at 104.14 120.65 180) (fields_autoplaced)
-    (effects (font (size 1.27 1.27)) (justify right bottom))
-  )
   (label "P19" (at 180.34 120.65 0) (fields_autoplaced)
