File: Hardware/2U-PCB-OBC_L476RG/OBC_L476RG/OBC_L476RG.kicad_sch (KiCad schematic)
At the start: 7 parts, among them J1 Bus Standard, J2 Micro_SD_Card_Det_Hirose_DM3AT, U2 NUCLEO_L476RG

Commit message: Project name was wrong in in kicad files. Project renamed
Connections:
- net +3.3V: no longer U2.16 (+3V3)
- net +5V: no longer names the net of U2.18 (+5V)
- no-connect marks 57 -> 59
Changed lines of the file:
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@@
   (junction (at 46.99 78.74) (diameter 0) (color 0 0 0 0)
   )
-  (junction (at 104.14 82.55) (diameter 0) (color 0 0 0 0)
-  )
   (junction (at 26.67 78.74) (diameter 0) (color 0 0 0 0)
-  )
-  (junction (at 105.41 66.04) (diameter 0) (color 0 0 0 0)
   )
   (junction (at 111.76 85.09) (diameter 0) (color 0 0 0 0)
@@
   (no_connect (at 162.56 97.79))
   (no_connect (at 226.06 72.39))
+  (no_connect (at 120.65 82.55))
   (no_connect (at 120.65 80.01))
   (no_connect (at 120.65 105.41))
@@
   (no_connect (at 120.65 133.35))
   (no_connect (at 120.65 123.19))
+  (no_connect (at 120.65 77.47))
   (no_connect (at 120.65 64.77))
   (no_connect (at 248.92 62.23))
@@
     (stroke (width 0) (type default))
   )
-  (wire (pts (xy 120.65 77.47) (xy 105.41 77.47))
-    (stroke (width 0) (type default))
-  )
   (wire (pts (xy 180.34 123.19) (xy 162.56 123.19))
     (stroke (width 0) (type default))
@@
     (stroke (width 0) (type default))
   )
-  (wire (pts (xy 120.65 82.55) (xy 104.14 82.55))
-    (stroke (width 0) (type default))
-  )
   (wire (pts (xy 180.34 120.65) (xy 162.56 120.65))
     (stroke (width 0) (type default))
@@
     (stroke (width 0) (type default))
   )
-  (wire (pts (xy 105.41 62.23) (xy 105.41 66.04))
-    (stroke (width 0) (type default))
-  )
   (wire (pts (xy 171.45 87.63) (xy 171.45 149.86))
     (stroke (width 0) (type default))
@@
     (stroke (width 0) (type default))
   )
-  (wire (pts (xy 104.14 82.55) (xy 100.33 82.55))
-    (stroke (width 0) (type default))
-  )
-  (wire (pts (xy 105.41 66.04) (xy 105.41 77.47))
-    (stroke (width 0) (type default))
-  )
   (wire (pts (xy 39.37 78.74) (xy 46.99 78.74))
     (stroke (width 0) (type default))
@@
   )
   (wire (pts (xy 222.25 102.87) (xy 226.06 102.87))
-    (stroke (width 0) (type default))
-  )
-  (wire (pts (xy 100.33 82.55) (xy 100.33 77.47))
     (stroke (width 0) (type default))
   )
@@
     (pin "2")
     (instances
-      (project "OBS_L476RG"
+      (project "OBC_L476RG"
         (path "/3074c2c6-4fd2-48c4-846c-d9e7f42bd5d3"
           (reference "C2") (unit 1)
@@
     (pin "1")
     (instances
-      (project "OBS_L476RG"
+      (project "OBC_L476RG"
         (path "/3074c2c6-4fd2-48c4-846c-d9e7f42bd5d3"
           (reference "#PWR06") (unit 1)
@@
     (pin "2")
     (instances
-      (project "OBS_L476RG"
+      (project "OBC_L476RG"
         (path "/3074c2c6-4fd2-48c4-846c-d9e7f42bd5d3"
           (reference "R1") (unit 1)
@@
         )
       )
-      (project "OBS_L476RG"
+      (project "OBC_L476RG"
         (path "/3074c2c6-4fd2-48c4-846c-d9e7f42bd5d3"
           (reference "J1") (unit 1)
@@
         (path "/4ae30ec6-0f79-4da8-b14c-df90c5069122"
           (reference "J3") (unit 1)
-        )
-      )
-    )
-  )
-  (symbol (lib_id "power:PWR_FLAG") (at 105.41 66.04 90) (unit 1)
-    (in_bom yes) (on_board yes) (dnp no) (fields_autoplaced)
-    (property "Reference" "#FLG01" (at 103.505 66.04 0)
-      (effects (font (size 1.27 1.27)) hide)
-    )
-    (property "Value" "PWR_FLAG" (at 101.6 66.04 90)
-      (effects (font (size 1.27 1.27)) (justify left))
-    )
-    (property "Footprint" "" (at 105.41 66.04 0)
-      (effects (font (size 1.27 1.27)) hide)
-    )
-    (property "Datasheet" "~" (at 105.41 66.04 0)
-      (effects (font (size 1.27 1.27)) hide)
-    )
-    (pin "1")
-    (instances
-      (project "OBS_L476RG"
-        (path "/3074c2c6-4fd2-48c4-846c-d9e7f42bd5d3"
-          (reference "#FLG01") (unit 1)
-        )
-      )
-    )
-  )
-  (symbol (lib_id "power:PWR_FLAG") (at 104.14 82.55 0) (unit 1)
-    (in_bom yes) (on_board yes) (dnp no) (fields_autoplaced)
-    (property "Reference" "#FLG02" (at 104.14 80.645 0)
-      (effects (font (size 1.27 1.27)) hide)
-    )
-    (property "Value" "PWR_FLAG" (at 104.14 77.47 0)
-      (effects (font (size 1.27 1.27)))
-    )
-    (property "Footprint" "" (at 104.14 82.55 0)
-      (effects (font (size 1.27 1.27)) hide)
-    )
-    (property "Datasheet" "~" (at 104.14 82.55 0)
-      (effects (font (size 1.27 1.27)) hide)
-    )
-    (pin "1")
-    (instances
-      (project "OBS_L476RG"
-        (path "/3074c2c6-4fd2-48c4-846c-d9e7f42bd5d3"
-          (reference "#FLG02") (unit 1)
         )
       )
@@
     (pin "9")
     (instances
-      (project "OBS_L476RG"
+      (project "OBC_L476RG"
         (path "/3074c2c6-4fd2-48c4-846c-d9e7f42bd5d3"
           (reference "J2") (unit 1)
@@
     (pin "1")
     (instances
-      (project "OBS_L476RG"
+      (project "OBC_L476RG"
         (path "/3074c2c6-4fd2-48c4-846c-d9e7f42bd5d3"
           (reference "#PWR04") (unit 1)
@@
     (pin "5")
     (instances
-      (project "OBS_L476RG"
+      (project "OBC_L476RG"
         (path "/3074c2c6-4fd2-48c4-846c-d9e7f42bd5d3"
           (reference "B1") (unit 1)
@@
     (pin "1")
     (instances
-      (project "OBS_L476RG"
+      (project "OBC_L476RG"
         (path "/3074c2c6-4fd2-48c4-846c-d9e7f42bd5d3"
           (reference "#PWR02") (unit 1)
@@
     (pin "1")
     (instances
-      (project "OBS_L476RG"
+      (project "OBC_L476RG"
         (path "/3074c2c6-4fd2-48c4-846c-d9e7f42bd5d3"
           (reference "#PWR09") (unit 1)
@@
     (pin "1")
     (instances
-      (project "OBS_L476RG"
+      (project "OBC_L476RG"
         (path "/3074c2c6-4fd2-48c4-846c-d9e7f42bd5d3"
           (reference "#PWR07") (unit 1)
@@
     (pin "1")
     (instances
-      (project "OBS_L476RG"
+      (project "OBC_L476RG"
         (path "/3074c2c6-4fd2-48c4-846c-d9e7f42bd5d3"
           (reference "#PWR03") (unit 1)
-        )
-      )
-    )
-  )
-  (symbol (lib_id "power:+3.3V") (at 105.41 62.23 0) (unit 1)
-    (in_bom yes) (on_board yes) (dnp no)
-    (property "Reference" "#PWR010" (at 105.41 66.04 0)
-      (effects (font (size 1.27 1.27)) hide)
-    )
-    (property "Value" "+3.3V" (at 105.41 57.15 0)
-      (effects (font (size 1.27 1.27)))
-    )
-    (property "Footprint" "" (at 105.41 62.23 0)
-      (effects (font (size 1.27 1.27)) hide)
-    )
-    (property "Datasheet" "" (at 105.41 62.23 0)
-      (effects (font (size 1.27 1.27)) hide)
-    )
-    (pin "1")
-    (instances
-      (project "OBS_L476RG"
-        (path "/3074c2c6-4fd2-48c4-846c-d9e7f42bd5d3"
-          (reference "#PWR010") (unit 1)
-        )
-      )
-    )
-  )
-  (symbol (lib_id "power:+5V") (at 100.33 77.47 0) (unit 1)
-    (in_bom yes) (on_board yes) (dnp no) (fields_autoplaced)
-    (property "Reference" "#PWR013" (at 100.33 81.28 0)
-      (effects (font (size 1.27 1.27)) hide)
-    )
-    (property "Value" "+5V" (at 100.33 72.39 0)
-      (effects (font (size 1.27 1.27)))
-    )
-    (property "Footprint" "" (at 100.33 77.47 0)
-      (effects (font (size 1.27 1.27)) hide)
-    )
-    (property "Datasheet" "" (at 100.33 77.47 0)
-      (effects (font (size 1.27 1.27)) hide)
-    )
-    (pin "1")
-    (instances
-      (project "OBS_L476RG"
-        (path "/3074c2c6-4fd2-48c4-846c-d9e7f42bd5d3"
-          (reference "#PWR013") (unit 1)
         )
       )
@@
     (pin "1")
     (instances
-      (project "OBS_L476RG"
+      (project "OBC_L476RG"
         (path "/3074c2c6-4fd2-48c4-846c-d9e7f42bd5d3"
           (reference "#PWR08") (unit 1)
@@
     (pin "2")
     (instances
-      (project "OBS_L476RG"
+      (project "OBC_L476RG"
         (path "/3074c2c6-4fd2-48c4-846c-d9e7f42bd5d3"
           (reference "C1") (unit 1)
@@
     (pin "1")
     (instances
-      (project "OBS_L476RG"
+      (project "OBC_L476RG"
         (path "/3074c2c6-4fd2-48c4-846c-d9e7f42bd5d3"
           (reference "#PWR01") (unit 1)
@@
     (pin "1")
     (instances
-      (project "OBS_L476RG"
+      (project "OBC_L476RG"
         (path "/3074c2c6-4fd2-48c4-846c-d9e7f42bd5d3"
           (reference "#PWR05") (unit 1)
@@
     (pin "33")
     (instances
-      (project "OBS_L476RG"
+      (project "OBC_L476RG"
         (path "/3074c2c6-4fd2-48c4-846c-d9e7f42bd5d3"
           (reference "U2") (unit 1)

Commit message: Some libraries were added for NAND gate. Also I2C in mikrobus changed. ROuting started respecting constraints.
Parts:
- B1: value ~ -> Buffer
- renumbered U2 to U1
Connections:
- net +3.3V: now also U1.16 (+3V3)
- no-connect marks 59 -> 58
Changed lines of the file:
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@@
   (junction (at 26.67 78.74) (diameter 0) (color 0 0 0 0)
+  )
+  (junction (at 30.48 20.32) (diameter 0) (color 0 0 0 0)
   )
   (junction (at 111.76 85.09) (diameter 0) (color 0 0 0 0)
@@
   (no_connect (at 120.65 133.35))
   (no_connect (at 120.65 123.19))
-  (no_connect (at 120.65 77.47))
   (no_connect (at 120.65 64.77))
   (no_connect (at 248.92 62.23))
@@
     (stroke (width 0) (type default))
   )
-  (wire (pts (xy 25.4 20.32) (xy 38.1 20.32))
+  (wire (pts (xy 25.4 20.32) (xy 30.48 20.32))
+    (stroke (width 0) (type default))
+  )
+  (wire (pts (xy 106.68 77.47) (xy 106.68 71.12))
     (stroke (width 0) (type default))
   )
@@
     (stroke (width 0) (type default))
   )
+  (wire (pts (xy 30.48 20.32) (xy 38.1 20.32))
+    (stroke (width 0) (type default))
+  )
   (wire (pts (xy 13.97 142.24) (xy 13.97 148.59))
     (stroke (width 0) (type default))
@@
   )
   (wire (pts (xy 222.25 102.87) (xy 226.06 102.87))
+    (stroke (width 0) (type default))
+  )
+  (wire (pts (xy 120.65 77.47) (xy 106.68 77.47))
     (stroke (width 0) (type default))
   )
@@
         (path "/3074c2c6-4fd2-48c4-846c-d9e7f42bd5d3"
           (reference "R1") (unit 1)
+        )
+      )
+    )
+  )
+  (symbol (lib_id "power:+3.3V") (at 106.68 71.12 0) (unit 1)
+    (in_bom yes) (on_board yes) (dnp no)
+    (property "Reference" "#PWR010" (at 106.68 74.93 0)
+      (effects (font (size 1.27 1.27)) hide)
+    )
+    (property "Value" "+3.3V" (at 106.68 66.04 0)
+      (effects (font (size 1.27 1.27)))
+    )
+    (property "Footprint" "" (at 106.68 71.12 0)
+      (effects (font (size 1.27 1.27)) hide)
+    )
+    (property "Datasheet" "" (at 106.68 71.12 0)
+      (effects (font (size 1.27 1.27)) hide)
+    )
+    (pin "1")
+    (instances
+      (project "OBC_L476RG"
+        (path "/3074c2c6-4fd2-48c4-846c-d9e7f42bd5d3"
+          (reference "#PWR010") (unit 1)
         )
       )
@@
   )
   (symbol (lib_id "SN74AHC1:SN74AHC1") (at 15.24 76.2 0) (unit 1)
-    (in_bom yes) (on_board yes) (dnp no) (fields_autoplaced)
-    (property "Reference" "B1" (at 18.415 73.66 0)
-      (effects (font (size 1.27 1.27)))
-    )
-    (property "Value" "~" (at 21.59 73.66 0)
+    (in_bom yes) (on_board yes) (dnp no)
+    (property "Reference" "B1" (at 19.05 73.66 0)
+      (effects (font (size 1.27 1.27)))
+    )
+    (property "Value" "Buffer" (at 18.7453 75.3734 0)
       (effects (font (size 1.27 1.27)))
     )
@@
     )
   )
+  (symbol (lib_id "power:PWR_FLAG") (at 30.48 20.32 0) (unit 1)
+    (in_bom yes) (on_board yes) (dnp no) (fields_autoplaced)
+    (property "Reference" "#FLG01" (at 30.48 18.415 0)
+      (effects (font (size 1.27 1.27)) hide)
+    )
+    (property "Value" "PWR_FLAG" (at 30.48 15.24 0)
+      (effects (font (size 1.27 1.27)))
+    )
+    (property "Footprint" "" (at 30.48 20.32 0)
+      (effects (font (size 1.27 1.27)) hide)
+    )
+    (property "Datasheet" "~" (at 30.48 20.32 0)
+      (effects (font (size 1.27 1.27)) hide)
+    )
+    (pin "1")
+    (instances
+      (project "OBC_L476RG"
+        (path "/3074c2c6-4fd2-48c4-846c-d9e7f42bd5d3"
+          (reference "#FLG01") (unit 1)
+        )
+      )
+    )
+  )
   (symbol (lib_id "power:+3.3V") (at 38.1 19.05 0) (unit 1)
     (in_bom yes) (on_board yes) (dnp no)
@@
   (symbol (lib_name "NUCLEO_L476RG_1") (lib_id "L476RG:NUCLEO_L476RG") (at 140.97 85.09 0) (unit 1)
     (in_bom yes) (on_board yes) (dnp no) (fields_autoplaced)
-    (property "Reference" "U2" (at 141.605 27.94 0)
+    (property "Reference" "U1" (at 141.605 27.94 0)
       (effects (font (size 1.27 1.27)))
     )
@@
       (project "OBC_L476RG"
         (path "/3074c2c6-4fd2-48c4-846c-d9e7f42bd5d3"
-          (reference "U2") (unit 1)
-        )
-      )
+          (reference "U1") (unit 1)
+        )
+      )
