File: Hardware/2U-PCB-Com_Nucleo-L432kC/Com_Nucleo-L432kc/Com_Nucleo-L432kc.kicad_sch (KiCad schematic)
At the start: 42 parts, among them IC1 PCI_EXPRESS_CARD, J1 Bus Standard, J2 I2C_Groove, J3 I2C_Groove, J4 Conn_01x08, J5 Conn_01x08, J6 Conn_01x15, J7 Conn_01x15, J8 I2C_Groove, J9 I2C_Groove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

Commit message: Traces almost ready, I'm avoiding through holes because it will be done in campus, not with specialized machines. Constraints: 125 um clearence and wire size. It will be not possible completly avoid through holes
Parts:
- removed R2: 100, Resistor_SMD:R_0402_1005Metric, symbol Device:R
- removed R9: 0, Resistor_SMD:R_0402_1005Metric, symbol Device:R
- added C13: 10u, Capacitor_SMD:C_0603_1608Metric, symbol Device:C
- added C14: 100n, Capacitor_SMD:C_0402_1005Metric, symbol Device:C
- added J10: Conn_01x01, Connector_PinSocket_1.27mm:PinSocket_1x01_P1.27mm_Vertical, symbol Connector_Generic:Conn_01x01
- J2, J3, J8, J9: value I2C_Groove -> I2C_Grove
- renumbered R3 to R2, R4 to R3, R5 to R4, R6 to R5, R7 to R6, R8 to R7
Connections:
- net +3V3: now also J6.14 (Pin_14), L432KC1.17 (+3V3), C13.1, C14.1
- net GND: now also C13.2, C14.2
- net L432KC_RESET: no longer J6.3 (Pin_3), L432KC1.28 (RESET)
- net TH1: now reaches IC1.6 (1.5V_2), R7.1
- net TH1: now also J10.1 (Pin_1)
- net AREF: now reaches J6.13 (Pin_13), L432KC1.18 (AREF)
- no-connect marks 46 -> 48
Other:
- note added: "Communication debug groves"
- note removed: "Communication debug grooves"
- moved on the sheet: C7, C8

Commit message: New library joined, cause we changed for a 7404 logic gate. All the routes were re-made.
Parts:
- removed C11: 10u, Capacitor_SMD:C_0603_1608Metric, symbol Device:C
- removed J10: Conn_01x01, Connector_PinSocket_1.27mm:PinSocket_1x01_P1.27mm_Vertical, symbol Connector_Generic:Conn_01x01
- removed JP4: Jumper_RESET_GPS_Open, Button_Switch_SMD:SW_Push_1P1T_NO_CK_KMR2, symbol Jumper:Jumper_2_Open
- removed U2: 74LVC2G02, SN74LVC2G02_SSOP:DCT8, symbol 74xGxx:74LVC2G02
- added U1: 7404, ul_SN74HC04N:N14, symbol 74xx_IEEE:7404
- C1, C13, C7, C9: footprint Capacitor_SMD:C_0603_1608Metric -> Capacitor_SMD:C_0805_2012Metric
- C10, C14, C2, C3, C4, C5, C6, C8: footprint Capacitor_SMD:C_0402_1005Metric -> Capacitor_SMD:C_0805_2012Metric
- C11: renamed from C12; footprint Capacitor_SMD:C_0402_1005Metric -> Capacitor_SMD:C_0805_2012Metric
- L432KC1: value ~ -> MCU
- R1, R2, R3, R4, R5, R6, R7: footprint Resistor_SMD:R_0402_1005Metric -> Resistor_SMD:R_0805_2012Metric
- renumbered JP5 to JP4
Connections:
- net +3V3: now also U1.14 (VCC), U1.14 (VCC); no longer B1.5 (VCC), J6.14 (Pin_14), L432KC1.17 (+3V3)
- net CS_MCU: now also U1.5
- net GND: now also U1.7 (GND), U1.7 (GND)
- net MCU_NRESET: now also U1.1
- net SX1303_RESET: now also U1.2
- net at B2.1 (OE): now also U1.6
- new net 3.3V: B1.5 (VCC), J6.14 (Pin_14), L432KC1.17 (+3V3)
Other:
- note added: "74LVC2G02 capacitors"
- note added: "CAN capacitors"
- note added: "Mikrobus capacitors"
- moved on the sheet: B2, C11, CR1, J4, J5, J6, J7, JP4, JP6, L432KC1

Commit message: The board is ready, need some revision
Parts:
- JP4: footprint Connector_PinHeader_1.27mm:PinHeader_1x02_P1.27mm_Vertical -> Connector_PinHeader_2.54mm:PinHeader_1x02_P2.54mm_Vertical
- JP5: renamed from JP6; footprint Connector_PinHeader_1.27mm:PinHeader_1x02_P1.27mm_Vertical -> Connector_PinHeader_2.54mm:PinHeader_1x02_P2.54mm_Vertical
Changed lines of the file:
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@@
       (effects (font (size 1.27 1.27)))
     )
-    (property "Footprint" "Connector_PinHeader_1.27mm:PinHeader_1x02_P1.27mm_Vertical" (at 50.165 140.335 0)
+    (property "Footprint" "Connector_PinHeader_2.54mm:PinHeader_1x02_P2.54mm_Vertical" (at 50.165 140.335 0)
       (effects (font (size 1.27 1.27)) hide)
     )
@@
   (symbol (lib_id "Jumper:Jumper_2_Open") (at 276.225 265.43 0) (unit 1)
     (in_bom yes) (on_board yes) (dnp no)
-    (property "Reference" "JP6" (at 276.225 259.08 0)
+    (property "Reference" "JP5" (at 276.225 259.08 0)
       (effects (font (size 1.27 1.27)))
     )
@@
       (effects (font (size 1.27 1.27)))
     )
-    (property "Footprint" "Connector_PinHeader_1.27mm:PinHeader_1x02_P1.27mm_Vertical" (at 276.225 265.43 0)
+    (property "Footprint" "Connector_PinHeader_2.54mm:PinHeader_1x02_P2.54mm_Vertical" (at 276.225 265.43 0)
       (effects (font (size 1.27 1.27)) hide)
     )
@@
       (project "Com_Nucleo-L432kc"
         (path "/0b43379d-830f-4a2c-bf01-7ac511af3f6d"
-          (reference "JP6") (unit 1)
+          (reference "JP5") (unit 1)
         )
       )
