File: Hardware/2U-PCB-Com_Nucleo-L432kC/Com_Nucleo-L432kc/Com_Nucleo-L432kc.kicad_sch (KiCad schematic)
At the start: 40 parts, among them IC1 PCI_EXPRESS_CARD, J1 Bus Standard, J2 I2C_Grove, J3 I2C_Grove, J4 Conn_01x08, J5 Conn_01x08, J6 Conn_01x15, J7 Conn_01x15, J8 I2C_Grove, J9 I2C_Grove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

Commit message: First version for fabrication
Other:
- moved on the sheet: CR1, J6, J7, JP5, L432KC1, U1A

Commit message: Flatsat connector was in the wrong side. All the routes were remade.
Connections:
- net +3V3: now also B1.5 (VCC)
- net 3.3V: no longer B1.5 (VCC)
- net RX_CALC: now also J7.7 (Pin_7), L432KC1.7 (D4); no longer J7.8 (Pin_8), L432KC1.8 (D5)
- net TX_CALC: now also J7.8 (Pin_8), L432KC1.8 (D5); no longer J7.7 (Pin_7), L432KC1.7 (D4)
Changed lines of the file:
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@@
     (effects (font (size 2 2)) (justify left bottom))
   )
-  (label "TX_CALC" (at 268.605 158.75 180) (fields_autoplaced)
+  (label "TX_CALC" (at 268.605 161.29 180) (fields_autoplaced)
     (effects (font (size 1.27 1.27)) (justify right bottom))
   )
@@
     (effects (font (size 1.27 1.27)) (justify right bottom))
   )
-  (label "RX_CALC" (at 268.605 161.29 180) (fields_autoplaced)
+  (label "RX_CALC" (at 268.605 158.75 180) (fields_autoplaced)
     (effects (font (size 1.27 1.27)) (justify right bottom))
   )
@@
   (label "CS_MCU" (at 50.165 263.525 180) (fields_autoplaced)
     (effects (font (size 1.27 1.27)) (justify right bottom))
-  )
-  (label "3.3V" (at 33.02 248.285 0) (fields_autoplaced)
-    (effects (font (size 1.27 1.27)) (justify left bottom))
   )
   (label "MKB_MISO" (at 330.2 91.44 180) (fields_autoplaced)
@@
         )
       )
+    )
+  )
+  (symbol (lib_id "power:+3.3V") (at 33.02 248.285 0) (unit 1)
+    (in_bom yes) (on_board yes) (dnp no)
+    (property "Reference" "#PWR09" (at 33.02 252.095 0)
+      (effects (font (size 1.27 1.27)) hide)
+    )
+    (property "Value" "+3.3V" (at 27.94 245.11 0)
+      (effects (font (size 1.27 1.27)))
+    )
+    (property "Footprint" "" (at 33.02 248.285 0)
+      (effects (font (size 1.27 1.27)) hide)
+    )
+    (property "Datasheet" "" (at 33.02 248.285 0)
+      (effects (font (size 1.27 1.27)) hide)
+    )
+    (pin "1")
+    (instances
+      (project "Com_Nucleo-L432kc"
+        (path "/0b43379d-830f-4a2c-bf01-7ac511af3f6d"
+          (reference "#PWR09") (unit 1)
+        )
+      )
+      (project "Corecell_Nucleo32"
+        (path "/4ae30ec6-0f79-4da8-b14c-df90c5069122"
+          (reference "#PWR0116") (unit 1)
+        )
+      )

Commit message: correction carte Lucas
Parts:
- removed JP1: Jumper_RESET_L432KC_Open, Button_Switch_SMD:SW_Push_1P1T_NO_CK_KMR2, symbol Jumper:Jumper_2_Open
- removed JP2: Jumper_MCU_Reset_Open, Button_Switch_SMD:SW_Push_1P1T_NO_CK_KMR2, symbol Jumper:Jumper_2_Open
- removed JP3: Jumper_SX1303_Reset_Open, Button_Switch_SMD:SW_Push_1P1T_NO_CK_KMR2, symbol Jumper:Jumper_2_Open
- added SW1: Jumper_RESET_L432KC_Open, Button_Switch_THT:SW_PUSH_6mm, symbol Switch:SW_Push
- added SW2: Jumper_MCU_Reset_Open, Button_Switch_THT:SW_PUSH_6mm, symbol Switch:SW_Push
- added SW3: Jumper_SX1303_Reset_Open, Button_Switch_THT:SW_PUSH_6mm, symbol Switch:SW_Push
- C1, C10, C11, C13, C14, C2, C3, C4, C5, C6, C7, C8, C9: footprint Capacitor_SMD:C_0805_2012Metric -> Capacitor_SMD:C_0805_2012Metric_Pad1.18x1.45mm_HandSolder
- CR1: footprint footprints:SO-8_STM -> Library:SO-8_STM
- J1: footprint flatsat_conn:flatsat_conn -> Library:flatsat_conn
- J4, J5: footprint Conn_mikro:MIkrobus_Connector -> Library:MIkrobus_Connector
- R1, R2, R3, R4, R5, R6, R7: footprint Resistor_SMD:R_0805_2012Metric -> Resistor_SMD:R_0805_2012Metric_Pad1.20x1.40mm_HandSolder
- U1: footprint ul_SN74HC04N:N14 -> Library:N14
Connections:
- net +3V3: now also SW3.2
- net GND: now also SW1.2, SW2.2
- net L432KC_RESET: now also SW1.1
- net MCU_NRESET: now also SW2.1
- net SX1303_RESET: now also SW3.1
