File: Hardware/2U-PCB-Com_Nucleo-L432kC/Com_Nucleo-L432kc/Projet Kicad/Com_Nucleo-L432kc.kicad_sch (KiCad schematic)
At the start: 40 parts, among them IC1 PCI_EXPRESS_CARD, J1 Bus Standard, J2 I2C_Grove, J3 I2C_Grove, J4 Conn_01x08, J5 Conn_01x08, J6 Conn_01x15, J7 Conn_01x15, J8 I2C_Grove, J9 I2C_Grove, SW1 Jumper_RESET_L432KC_Open, SW2 Jumper_MCU_Reset_Open, SW3 Jumper_SX1303_Reset_Open, U1 7404

Commit message: début de la reprise de la carte
Parts:
- removed B1, B2: SN74AHC1G125DBVT, Package_SO:TSOP-5_1.65x3.05mm_P0.95mm, symbol SN74AHC1:SN74AHC1
- removed C11: 100n, Capacitor_SMD:C_0805_2012Metric_Pad1.18x1.45mm_HandSolder, symbol Device:C
- removed J2: I2C_Grove, Connector_PinSocket_2.54mm:PinSocket_1x04_P2.54mm_Vertical, symbol Connector_Generic:Conn_01x04
- removed J4, J5: Conn_01x08, Library:MIkrobus_Connector, symbol Connector_Generic:Conn_01x08
- removed JP4: Jumper_STANDBY_GPS_Open, Connector_PinHeader_2.54mm:PinHeader_1x02_P2.54mm_Vertical, symbol Jumper:Jumper_2_Open
- removed SW2: Jumper_MCU_Reset_Open, Button_Switch_THT:SW_PUSH_6mm, symbol Switch:SW_Push
- removed SW3: Jumper_SX1303_Reset_Open, Button_Switch_THT:SW_PUSH_6mm, symbol Switch:SW_Push
- removed U1: 7404, Library:N14, symbol 74xx_IEEE:7404
- added J3: I2C_Grove, Connector:NS-Tech_Grove_1x04_P2mm_Vertical, symbol Connector_Generic:Conn_01x04
- added J5: MIKROE-4247, MIKROE4247, symbol Com_L432KC_symbols:MIKROE-4247
- added JP1: PWM1_SEL, symbol Jumper:Jumper_3_Open
- added U1: STTS751, SON65P200X200X55-6N, symbol Com_L432KC_symbols:STTS751-0DP3F
- R1, R2: value 0 -> 4K7; footprint Resistor_SMD:R_0805_2012Metric_Pad1.20x1.40mm_HandSolder -> (none)
- R3: value 100 -> 4K7; footprint Resistor_SMD:R_0805_2012Metric_Pad1.20x1.40mm_HandSolder -> (none)
- R4: value 100 -> 47K; footprint Resistor_SMD:R_0805_2012Metric_Pad1.20x1.40mm_HandSolder -> (none)
- R5: value 100 -> 7K5; footprint Resistor_SMD:R_0805_2012Metric_Pad1.20x1.40mm_HandSolder -> (none)
- R6: value 100 -> 0; footprint Resistor_SMD:R_0805_2012Metric_Pad1.20x1.40mm_HandSolder -> (none)
- R7: footprint Resistor_SMD:R_0805_2012Metric_Pad1.20x1.40mm_HandSolder -> (none)
- SW1: value Jumper_RESET_L432KC_Open -> Reset
- renumbered C6 to C10, C7 to C11, C8 to C13, C13 to C2, C2 to C3, C14 to C4, C3 to C5, C4 to C6, C9 to C7, C5 to C8, C10 to C9, J7 to J2, J3 to J4, J8 to J6, J6 to J7, JP5 to JP2
Connections:
- net 3.3V is gone; now on an unnamed net: J7.14 (Pin_14), L432KC1.17 (+3V3)
- net HOST_MISO is gone; now on net +3V3: R4.1
- net SX1303_RESET is gone; now on net RST_LORA_CORE: IC1.22 (~{PERST})
- net +3V3: now also C11.1, C13.1, R1.1, R2.1, R3.1, R5.2, J3.3 (Pin_3), U1.3 (VDD)
- net GND: now also J3.4 (Pin_4), J5.1 (GND_1), J5.16 (GND_2), U1.5 (GND)
- net MISO: now also IC1.47 (RESERVED2), J2.15 (Pin_15), L432KC1.15 (D12), J5.14 (MOSI); no longer J7.7 (Pin_7), L432KC1.24 (A5)
- net SCL: now also R2.2, J3.1 (Pin_1), J5.4 (SCL), U1.1 (SCL); no longer IC1.30 (SMB_SCL)
- net SDA: now also R3.2, J3.2 (Pin_2), J5.3 (SDA), U1.6 (SDA); no longer IC1.32 (SMB_SDA)
- net at R6.2: no longer IC1.51 (RESERVED4)
- net at IC1.23 (PERn0): no longer R2.2
- net at IC1.13 (REFCLK+): no longer R1.2
- net +5V: now reaches J1.4 (5V)
- net +5V: now also J1.3 (V_IN), R7.1, J5.2 (+5V)
- net SCLK: now reaches IC1.45 (RESERVED1)
- net SCLK: now also J7.15 (Pin_15), L432KC1.16 (D13), J5.12 (SCK); no longer R3.2
- net at R4.2: now also U1.2 (~{EVENT}); no longer IC1.47 (RESERVED2)
- net MOSI: now reaches IC1.49 (RESERVED3)
- net MOSI: now also J2.14 (Pin_14), L432KC1.14 (D11), J5.13 (MISO); no longer R5.2
- net at J7.3 (Pin_3): now also L432KC1.28 (RESET)
- net at J7.4 (Pin_4), L432KC1.27 (+5V): now also R7.2
- net at J2.10 (Pin_10): now also L432KC1.10 (D7)
- net at J2.11 (Pin_11): now also L432KC1.11 (D8)
- net AN renamed GPIO6_SX1303
- net GPIO6_SX1303: now also IC1.6 (1.5V_2)
- net CAN1_RX renamed CAN_RX
- net CAN1_TX renamed CAN_TX
- removed net CS_MCU: J2.15 (Pin_15), L432KC1.15 (D12), R6.1
- net GPIO(6) renamed UART_RX_INISAT
- net UART_RX_INISAT: now also J1.17 (RX/SDA); no longer R7.2
- net HOST_SCK renamed SENS1
- net SENS1: now also J1.8 (NC3); no longer R3.1
- net INT_MKR renamed UART_TX_INISAT
- net UART_TX_INISAT: now also J1.19 (TX/SCL)
- net L432KC_RESET renamed RESET_GENERAL
- net RESET_GENERAL: now also R1.2, J5.10 (RST)
- net MCU_MOSI renamed INT_MK
- net INT_MK: now also J5.7 (INT); no longer R5.1
- removed net MCU_NRESET: J2.14 (Pin_14), L432KC1.14 (D11), R1.1, R2.1
- net PWM_MAG-Y renamed RST_LORA_CORE
- net RST_LORA_CORE: no longer J1.9 (NC4)
- net PWM_MKR renamed CS_LORA_CORE
- net CS_LORA_CORE: now also IC1.51 (RESERVED4)
- net PWM_ROUE/MAG-X renamed PWM1
- net PWM1: now also JP1.2 (C); no longer J1.6 (NC1)
- net RESET_SIGNAL renamed CS_MK
- net CS_MK: now also J5.11 (CS); no longer J1.30 (PWM_O_1)
- net RX_CALC renamed UART_RX_MK
- net UART_RX_MK: now also J5.6 (RX); no longer J1.17 (RX/SDA)
- removed net SENS_MAG-Y: J1.11 (NC), J7.15 (Pin_15), L432KC1.16 (D13)
- net SENS_ROUE/MAG-X renamed SENS2
- net SENS2: now also J1.11 (NC); no longer J1.8 (NC3)
- net STANDBY_GPS: no longer names the net of IC1.25 (PERp0)
- removed net TH1: IC1.6 (1.5V_2), R7.1
- net TX_CALC renamed UART_TX_MK
- net UART_TX_MK: now also J5.5 (TX); no longer J1.19 (TX/SCL)
- removed net Vin: C11.1, C13.1, J1.3 (V_IN), J7.1 (Pin_1), L432KC1.30 (VIN)
- new net: R5.1, U1.4 (ADDR/~{THERM})
- new net: J7.1 (Pin_1), L432KC1.30 (VIN)
- new net +3.3V: J5.15 (+3.3V), R6.1
- new net PWM2: J1.9 (NC4), J7.7 (Pin_7), L432KC1.24 (A5)
- new net PWM_INISAT: J1.6 (NC1), JP1.1 (A)
- new net PWM_MK: J5.8 (PWM), JP1.3 (B)
- no-connect marks 48 -> 45
Other:
- note added: "Addresse i2c : 0x48"
- note added: "Capteur de température"
- note added: "Connecteur Inisat"
- note added: "Jumpers"
- note added: "Selection de l'alimentation 3.3V ou 5V avec R6 et R7 ==> ATTENTION: ne pas monter les deux résistances !"
- note added: "VIN = 5V d'après le schema de la carte alim"
- note added: "i2c pull-up (ne monter que si necessaire)"
- note removed: "74LVC2G02 capacitors"
- note removed: "Power source and UART communication (Calculatrice)"
- moved on the sheet: C1, C10, C11, C13, C2, C3, C4, C5, C6, C7, C8, C9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
