File: Hardware/2U-PCB-Com_Nucleo-L432kC/Com_Nucleo-L432kc/Projet Kicad/Com_Nucleo-L432kc.kicad_sch (KiCad schematic)
At the start: 34 parts, among them IC1 PCI_EXPRESS_CARD, J1 Bus Standard, J2 Conn_01x15, J3 I2C_Grove, J4 I2C_Grove, J5 MIKROE-4247, J6 I2C_Grove, J7 Conn_01x15, J9 I2C_Grove, SW1 Reset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

Commit message: schématique terminée
Parts:
- added JP3: RX_SEL, symbol Jumper:Jumper_3_Open
- added JP4: TX_SEL, symbol Jumper:Jumper_3_Open
- added JP5: INT_SEL, symbol Jumper:Jumper_3_Open
- added R8, R9: 0, symbol Device:R
Connections:
- net +3.3V: now also R8.1
- net +3V3: no longer CR1.3 (VS)
- net +5V: now also R9.1
- net INT_MK: now also JP5.3 (B); no longer J7.6 (Pin_6), L432KC1.25 (A6)
- net PPS_LORA_CORE: now also JP5.1 (A)
- net UART_RX_1: now also JP3.2 (C)
- net UART_RX_LORA_CORE: now also IC1.33 (PETp0), JP4.1 (A); no longer IC1.31 (PETn0)
- net UART_RX_MK: now also JP4.3 (B)
- net UART_TX_1: now also JP4.2 (C)
- net UART_TX_LORA_CORE: now also IC1.31 (PETn0), JP3.1 (A); no longer IC1.33 (PETp0)
- net UART_TX_MK: now also JP3.3 (B)
- new net: CR1.3 (VS), R8.2, R9.2
- new net INT1: J7.6 (Pin_6), JP5.2 (C), L432KC1.25 (A6)
Other:
- moved on the sheet: CR1, J4, J6, J9, JP1, JP2

Commit message: routage terminé
Parts:
- removed C11: 10u, Capacitor_SMD:C_0805_2012Metric_Pad1.18x1.45mm_HandSolder, symbol Device:C
- removed C13: 100n, Capacitor_SMD:C_0805_2012Metric_Pad1.18x1.45mm_HandSolder, symbol Device:C
- removed J3: I2C_Grove, Connector:NS-Tech_Grove_1x04_P2mm_Vertical, symbol Connector_Generic:Conn_01x04
- removed R4: 47K, symbol Device:R
- removed R5: 7K5, symbol Device:R
- removed U1: STTS751, SON65P200X200X55-6N, symbol Com_L432KC_symbols:STTS751-0DP3F
- added R10, R11, R12, R13, R14, R15: 0, Resistor_SMD:R_0805_2012Metric_Pad1.20x1.40mm_HandSolder, symbol Device:R
- added U2: MCP9808_MSOP, Package_SO:MSOP-8_3x3mm_P0.65mm, symbol Sensor_Temperature:MCP9808_MSOP
- CR1: footprint Library:SO-8_STM -> Package_SO:SO-8_3.9x4.9mm_P1.27mm
- J1: footprint Library:flatsat_conn -> Com_L432KC_footprint:flatsat_conn
- J5: footprint MIKROE4247 -> Com_L432KC_footprint:MIKROE4247
- JP1, JP3, JP4, JP5: footprint (none) -> Connector_PinHeader_1.27mm:PinHeader_1x03_P1.27mm_Vertical
- R1, R2, R3, R6, R7, R8, R9: footprint (none) -> Resistor_SMD:R_0805_2012Metric_Pad1.20x1.40mm_HandSolder
Connections:
- net +3.3V is gone; now on net +3V3: J5.15 (+3.3V), R6.1, R8.1
- net +3V3: now also R11.1, R12.1, R14.1, U2.8 (V_{DD}); no longer C7.1, C9.1
- net GND: now also R10.1, R13.1, R15.1, U2.4 (GND)
- net SCL: now also U2.2 (SCL)
- net SDA: now also U2.1 (SDA)
- net at CR1.3 (VS), R8.2, R9.2: now also C7.1, C9.1
- new net: R10.2, R11.2, U2.7 (A0)
- new net: R14.2, R15.2, U2.5 (A2)
- new net: R12.2, R13.2, U2.6 (A1)
- no-connect marks 42 -> 43
Other:
- note added: "Addresse i2c : 0b0011 A2 A1 A0"
- note added: "PWM"
- note removed: "Addresse i2c : 0x48"
- note removed: "CAN capacitors"
- note removed: "Decoupling and bolt capacitors for Nucleo"
- moved on the sheet: C7, C9, CR1, J4, J5, J6, J9, JP2, R8, R9

Commit message: ajout documentation
Parts:
- added R4: 4K7, Resistor_SMD:R_0805_2012Metric_Pad1.20x1.40mm_HandSolder, symbol Device:R
- J2, J7: footprint Connector_PinSocket_2.54mm:PinSocket_1x15_P2.54mm_Vertical -> Connector_PinHeader_2.54mm:PinHeader_1x15_P2.54mm_Vertical
Connections:
- net +3V3: now also R4.1; no longer JP2.2 (B)
- net GND: now also JP2.2 (B)
- net at CR1.8 (ASC), JP2.1 (A): now also R4.2
Other:
- moved on the sheet: JP2
Changed lines of the file:
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@@
 	)
 	(junction
+		(at 367.03 227.33)
+		(diameter 0)
+		(color 0 0 0 0)
+	)
+	(junction
 		(at 124.46 248.92)
 		(diameter 0)
@@
 	(wire
 		(pts
-			(xy 373.38 231.14) (xy 373.38 229.87)
-		)
-		(stroke
-			(width 0)
-			(type default)
-		)
-	)
-	(wire
-		(pts
 			(xy 48.26 40.64) (xy 48.26 44.45)
 		)
@@
 	(wire
 		(pts
+			(xy 393.7 227.33) (xy 391.16 227.33)
+		)
+		(stroke
+			(width 0)
+			(type default)
+		)
+	)
+	(wire
+		(pts
 			(xy 68.58 243.84) (xy 68.58 246.38)
 		)
@@
 	(wire
 		(pts
-			(xy 394.97 227.33) (xy 383.54 227.33)
-		)
-		(stroke
-			(width 0)
-			(type default)
-		)
-	)
-	(wire
-		(pts
 			(xy 68.58 243.84) (xy 78.74 243.84)
 		)
@@
 	(wire
 		(pts
+			(xy 364.49 232.41) (xy 367.03 232.41)
+		)
+		(stroke
+			(width 0)
+			(type default)
+		)
+	)
+	(wire
+		(pts
 			(xy 322.58 213.36) (xy 316.23 213.36)
 		)
@@
 	(wire
 		(pts
-			(xy 377.19 231.14) (xy 373.38 231.14)
+			(xy 318.77 229.87) (xy 318.77 240.03)
 		)
 		(stroke
@@
 	(wire
 		(pts
-			(xy 318.77 229.87) (xy 318.77 240.03)
+			(xy 60.96 264.16) (xy 78.74 264.16)
 		)
 		(stroke
@@
 	(wire
 		(pts
-			(xy 60.96 264.16) (xy 78.74 264.16)
+			(xy 336.55 212.09) (xy 332.74 212.09)
 		)
 		(stroke
@@
 	(wire
 		(pts
-			(xy 336.55 212.09) (xy 332.74 212.09)
+			(xy 393.7 227.33) (xy 393.7 234.95)
 		)
 		(stroke
@@
 	(wire
 		(pts
+			(xy 364.49 229.87) (xy 367.03 229.87)
+		)
+		(stroke
+			(width 0)
+			(type default)
+		)
+	)
+	(wire
+		(pts
 			(xy 82.55 44.45) (xy 82.55 40.64)
 		)
@@
 	(wire
 		(pts
-			(xy 364.49 227.33) (xy 373.38 227.33)
+			(xy 364.49 227.33) (xy 367.03 227.33)
 		)
 		(stroke
@@
 	(wire
 		(pts
-			(xy 372.11 232.41) (xy 364.49 232.41)
-		)
-		(stroke
-			(width 0)
-			(type default)
-		)
-	)
-	(wire
-		(pts
 			(xy 124.46 203.2) (xy 124.46 220.98)
 		)
@@
 	(wire
 		(pts
-			(xy 377.19 233.68) (xy 372.11 233.68)
+			(xy 130.81 228.6) (xy 130.81 264.16)
 		)
 		(stroke
@@
 	(wire
 		(pts
-			(xy 130.81 228.6) (xy 130.81 264.16)
+			(xy 53.34 135.89) (xy 53.34 134.62)
 		)
 		(stroke
@@
 	(wire
 		(pts
-			(xy 53.34 135.89) (xy 53.34 134.62)
+			(xy 340.36 137.16) (xy 379.73 137.16)
 		)
 		(stroke
@@
 	(wire
 		(pts
-			(xy 340.36 137.16) (xy 379.73 137.16)
+			(xy 181.61 138.43) (xy 182.88 138.43)
 		)
 		(stroke
@@
 	(wire
 		(pts
-			(xy 181.61 138.43) (xy 182.88 138.43)
+			(xy 257.81 227.33) (xy 250.19 227.33)
 		)
 		(stroke
@@
 	(wire
 		(pts
-			(xy 257.81 227.33) (xy 250.19 227.33)
+			(xy 53.34 134.62) (xy 53.34 132.08)
 		)
 		(stroke
@@
 	(wire
 		(pts
-			(xy 53.34 134.62) (xy 53.34 132.08)
+			(xy 367.03 227.33) (xy 381 227.33)
 		)
 		(stroke
@@
 	(wire
 		(pts
-			(xy 394.97 224.79) (xy 394.97 227.33)
-		)
-		(stroke
-			(width 0)
-			(type default)
-		)
-	)
-	(wire
-		(pts
 			(xy 71.12 29.21) (xy 82.55 29.21)
 		)
@@
 	(wire
 		(pts
-			(xy 373.38 229.87) (xy 364.49 229.87)
-		)
-		(stroke
-			(width 0)
-			(type default)
-		)
-	)
-	(wire
-		(pts
 			(xy 382.27 40.64) (xy 378.46 40.64)
 		)
@@
 	(wire
 		(pts
-			(xy 372.11 233.68) (xy 372.11 232.41)
-		)
-		(stroke
-			(width 0)
-			(type default)
-		)
-	)
-	(wire
-		(pts
 			(xy 213.36 38.1) (xy 208.28 38.1)
 		)
@@
 	)
 	(label "CAN_TD"
-		(at 377.19 231.14 0)
+		(at 367.03 229.87 0)
 		(fields_autoplaced yes)
 		(effects
@@
 	)
 	(label "CAN_RD"
-		(at 377.19 233.68 0)
+		(at 367.03 232.41 0)
 		(fields_autoplaced yes)
 		(effects
@@
 	(symbol
 		(lib_id "power:+3.3V")
-		(at 394.97 224.79 0)
+		(at 367.03 219.71 0)
 		(unit 1)
 		(exclude_from_sim no)
@@
 		(fields_autoplaced yes)
 		(property "Reference" "#PWR031"
-			(at 394.97 228.6 0)
+			(at 367.03 223.52 0)
 			(effects
 				(font
@@
 		)
 		(property "Value" "+3V3"
-			(at 394.97 219.71 0)
+			(at 367.03 214.63 0)
 			(effects
 				(font
@@
 		)
 		(property "Footprint" ""
-			(at 394.97 224.79 0)
+			(at 367.03 219.71 0)
 			(effects
 				(font
@@
 		)
 		(property "Datasheet" ""
-			(at 394.97 224.79 0)
+			(at 367.03 219.71 0)
 			(effects
 				(font
@@
 		)
 		(property "Description" ""
-			(at 394.97 224.79 0)
+			(at 367.03 219.71 0)
 			(effects
 				(font
@@
 			)
 		)
-		(property "Footprint" "Connector_PinSocket_2.54mm:PinSocket_1x15_P2.54mm_Vertical"
+		(property "Footprint" "Connector_PinHeader_2.54mm:PinHeader_1x15_P2.54mm_Vertical"
 			(at 384.81 142.24 0)
 			(effects
@@
 	)
 	(symbol
+		(lib_id "Device:R")
+		(at 367.03 223.52 0)
+		(unit 1)
+		(exclude_from_sim no)
+		(in_bom yes)
+		(on_board yes)
+		(dnp no)
+		(fields_autoplaced yes)
+		(property "Reference" "R4"
+			(at 369.57 222.2499 0)
+			(effects
+				(font
+					(size 1.27 1.27)
+				)
+				(justify left)
+			)
+		)
+		(property "Value" "4K7"
+			(at 369.57 224.7899 0)
+			(effects
+				(font
+					(size 1.27 1.27)
+				)
+				(justify left)
+			)
+		)
+		(property "Footprint" "Resistor_SMD:R_0805_2012Metric_Pad1.20x1.40mm_HandSolder"
+			(at 365.252 223.52 90)
+			(effects
+				(font
+					(size 1.27 1.27)
+				)
+				(hide yes)
+			)
+		)
+		(property "Datasheet" "~"
+			(at 367.03 223.52 0)
+			(effects
+				(font
+					(size 1.27 1.27)
+				)
+				(hide yes)
+			)
+		)
+		(property "Description" "Resistor"
+			(at 367.03 223.52 0)
+			(effects
+				(font
+					(size 1.27 1.27)
+				)
+				(hide yes)
+			)
+		)
+		(pin "1"
+		)
+		(pin "2"
+		)
+		(instances
+			(project "Com_Nucleo-L432kc"
+				(path "/0b43379d-830f-4a2c-bf01-7ac511af3f6d"
+					(reference "R4")
+					(unit 1)
+				)
+			)
+		)
+	)
+	(symbol
 		(lib_id "Device:C")
 		(at 36.83 36.83 0)
@@
 			)
 		)
-		(property "Footprint" "Connector_PinSocket_2.54mm:PinSocket_1x15_P2.54mm_Vertical"
+		(property "Footprint" "Connector_PinHeader_2.54mm:PinHeader_1x15_P2.54mm_Vertical"
 			(at 266.7 142.24 0)
 			(effects
@@
 	(symbol
 		(lib_id "Jumper:Jumper_2_Open")
-		(at 378.46 227.33 0)
+		(at 386.08 227.33 0)
 		(unit 1)
 		(exclude_from_sim no)
@@
 		(dnp no)
 		(property "Reference" "JP2"
-			(at 378.46 220.98 0)
+			(at 386.08 220.98 0)
 			(effects
 				(font
@@
 		)
 		(property "Value" "speed_controller"
-			(at 378.46 223.52 0)
+			(at 386.08 223.52 0)
 			(effects
 				(font
@@
 		)
 		(property "Footprint" "Connector_PinHeader_2.54mm:PinHeader_1x02_P2.54mm_Vertical"
-			(at 378.46 227.33 0)
+			(at 386.08 227.33 0)
 			(effects
 				(font
@@
 		)
 		(property "Datasheet" "~"
-			(at 378.46 227.33 0)
+			(at 386.08 227.33 0)
 			(effects
 				(font
@@
 		)
 		(property "Description" ""
-			(at 378.46 227.33 0)
+			(at 386.08 227.33 0)
 			(effects
 				(font
@@
 					(unit 1)
 				)
+			)
+		)
+	)
+	(symbol
+		(lib_id "power:GND")
+		(at 393.7 234.95 0)
+		(unit 1)
+		(exclude_from_sim no)
+		(in_bom yes)
+		(on_board yes)
+		(dnp no)
+		(fields_autoplaced yes)
+		(property "Reference" "#PWR011"
+			(at 393.7 241.3 0)
+			(effects
+				(font
+					(size 1.27 1.27)
+				)
+				(hide yes)
+			)
+		)
+		(property "Value" "GND"
+			(at 393.7 240.03 0)
+			(effects
+				(font
+					(size 1.27 1.27)
+				)
+			)
+		)
+		(property "Footprint" ""
+			(at 393.7 234.95 0)
+			(effects
+				(font
+					(size 1.27 1.27)
+				)
+				(hide yes)
+			)
+		)
+		(property "Datasheet" ""
+			(at 393.7 234.95 0)
+			(effects
+				(font
+					(size 1.27 1.27)
+				)
+				(hide yes)
+			)
+		)
+		(property "Description" ""
+			(at 393.7 234.95 0)
+			(effects
+				(font
+					(size 1.27 1.27)
+				)
+				(hide yes)
+			)
+		)
+		(pin "1"
+		)
+		(instances
+			(project "Com_Nucleo-L432kc"
+				(path "/0b43379d-830f-4a2c-bf01-7ac511af3f6d"
+					(reference "#PWR011")
+					(unit 1)
+				)

Commit message: ajout documentation bis
Parts:
- JP1, JP3, JP4, JP5: footprint Connector_PinHeader_1.27mm:PinHeader_1x03_P1.27mm_Vertical -> Connector_PinHeader_2.54mm:PinHeader_1x03_P2.54mm_Vertical
Changed lines of the file:
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@@
 			)
 		)
-		(property "Footprint" "Connector_PinHeader_1.27mm:PinHeader_1x03_P1.27mm_Vertical"
+		(property "Footprint" "Connector_PinHeader_2.54mm:PinHeader_1x03_P2.54mm_Vertical"
 			(at 167.64 138.43 0)
 			(effects
@@
 			)
 		)
-		(property "Footprint" "Connector_PinHeader_1.27mm:PinHeader_1x03_P1.27mm_Vertical"
+		(property "Footprint" "Connector_PinHeader_2.54mm:PinHeader_1x03_P2.54mm_Vertical"
 			(at 189.23 138.43 0)
 			(effects
@@
 			)
 		)
-		(property "Footprint" "Connector_PinHeader_1.27mm:PinHeader_1x03_P1.27mm_Vertical"
+		(property "Footprint" "Connector_PinHeader_2.54mm:PinHeader_1x03_P2.54mm_Vertical"
 			(at 144.78 138.43 0)
 			(effects
@@
 			)
 		)
-		(property "Footprint" "Connector_PinHeader_1.27mm:PinHeader_1x03_P1.27mm_Vertical"
+		(property "Footprint" "Connector_PinHeader_2.54mm:PinHeader_1x03_P2.54mm_Vertical"
 			(at 105.41 130.81 0)
 			(effects

Commit message: finalisation Thingsat Inisat v1.0
Connections:
- net MISO: now also J5.13 (MISO); no longer J5.14 (MOSI)
- net MOSI: now also J5.14 (MOSI); no longer J5.13 (MISO)
Changed lines of the file:
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@@
 	)
 	(label "MOSI"
-		(at 330.2 78.74 180)
+		(at 330.2 81.28 180)
 		(fields_autoplaced yes)
 		(effects
@@
 	)
 	(label "MISO"
-		(at 330.2 81.28 180)
-		(fields_autoplaced yes)
-		(effects
+		(at 330.2 78.74 180)
+		(fields_autoplaced yes)
+		(effects
