File: Hardware/2U-PCB-Com_Nucleo-L432kC/Com_Nucleo-L432kc/Projet Kicad/_autosave-Com_Nucleo-L432kc.kicad_sch (KiCad schematic)
At the start: 34 parts, among them IC1 PCI_EXPRESS_CARD, J1 Bus Standard, J2 Conn_01x15, J3 I2C_Grove, J4 I2C_Grove, J5 MIKROE-4247, J6 I2C_Grove, J7 Conn_01x15, J9 I2C_Grove, SW1 Reset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

Commit message: schématique terminée
Parts:
- added JP3: RX_SEL, symbol Jumper:Jumper_3_Open
- added JP4: TX_SEL, symbol Jumper:Jumper_3_Open
- added JP5: INT_SEL, symbol Jumper:Jumper_3_Open
Connections:
- net INT_MK: now also JP5.3 (B); no longer J7.6 (Pin_6), L432KC1.25 (A6)
- net PPS_LORA_CORE: now also JP5.1 (A)
- net UART_RX_1: now also JP3.2 (C)
- net UART_RX_LORA_CORE: now also IC1.33 (PETp0), JP4.1 (A); no longer IC1.31 (PETn0)
- net UART_RX_MK: now also JP4.3 (B)
- net UART_TX_1: now also JP4.2 (C)
- net UART_TX_LORA_CORE: now also IC1.31 (PETn0), JP3.1 (A); no longer IC1.33 (PETp0)
- net UART_TX_MK: now also JP3.3 (B)
- new net INT1: J7.6 (Pin_6), JP5.2 (C), L432KC1.25 (A6)
Other:
- moved on the sheet: CR1, J4, J6, J9, JP1
